Commit message: Build with catkin.

File: tests/files/combined.urdf.xacro (robot description, xacro)
@@ -1,3 +1,3 @@
-<?xml version="1.0" ?>
+<?xml version="1.0" encoding="utf-8"?>
 <robot name="combined" xmlns:xacro="http://www.ros.org/wiki/xacro">
   <xacro:include filename="threelink.urdf.xacro" />

File: tests/files/tool2.urdf (robot description, URDF)
Before this commit: robot tool, 1 links, 1 joints
Links:
- link tool: mass $(arg mass) -> 2
