Commit message: Add test for localizing assets.

File: tests/files/xacro/mesh2.urdf.xacro (robot description, xacro)
@@ -5,5 +5,5 @@
       <origin rpy="0 0 0" xyz="0 0 0"/>
       <geometry>
-        <mesh filename="package://xacrodoc/tests/files/assets/fakemesh.txt"/>
+        <mesh filename="package://xacrodoc/tests/files/assets/one/fakemesh.txt"/>
       </geometry>
       <material name="black"/>
@@ -12,5 +12,5 @@
       <origin rpy="0 0 0" xyz="0 0 0"/>
       <geometry>
-        <cylinder length="0.15" radius="0.02"/>
+        <mesh filename="package://xacrodoc/tests/files/assets/two/fakemesh.txt"/>
       </geometry>
     </collision>
