Commit message: Heavily revise the MJCF API.

File: tests/files/xacro/mesh.urdf.xacro (robot description, xacro)
@@ -2,15 +2,8 @@
 <robot name="mesh" xmlns:xacro="http://wiki.ros.org/xacro">
   <link name="mesh">
-    <visual>
-      <origin rpy="0 0 0" xyz="0 0 0"/>
-      <geometry>
-        <mesh filename="package://xacrodoc/tests/files/assets/fakemesh.txt"/>
-      </geometry>
-      <material name="black"/>
-    </visual>
     <collision>
       <origin rpy="0 0 0" xyz="0 0 0"/>
       <geometry>
-        <cylinder length="0.15" radius="0.02"/>
+        <mesh filename="package://xacrodoc/tests/files/assets/base.stl"/>
       </geometry>
     </collision>

File: tests/files/xacro/mesh2.urdf.xacro (robot description, xacro)
@@ -5,5 +5,5 @@
       <origin rpy="0 0 0" xyz="0 0 0"/>
       <geometry>
-        <mesh filename="package://xacrodoc/tests/files/assets/one/fakemesh.txt"/>
+        <mesh filename="package://xacrodoc/tests/files/assets/one/base.stl"/>
       </geometry>
       <material name="black"/>
@@ -12,5 +12,5 @@
       <origin rpy="0 0 0" xyz="0 0 0"/>
       <geometry>
-        <mesh filename="package://xacrodoc/tests/files/assets/two/fakemesh.txt"/>
+        <mesh filename="package://xacrodoc/tests/files/assets/two/base.stl"/>
       </geometry>
     </collision>
